File: eagle/apple-idun.sch (EAGLE design)
At the start: 9 parts, among them J1 USBMICROB, U1 FT240XQ, U2 TPS2082D

Commit message: Add multiple sheets; finalize FIFO and load switch
Parts:
- added R3, R4: 100K, rcl:R-US_R0805
- U1: value FT240XQ -> FT240XS; device apple-idun:FT240XQ -> apple-idun:FT240XS
Connections:
- net D0 renamed FIFO_DATA0
- net D1 renamed FIFO_DATA1
- net D2 renamed FIFO_DATA2
- net D3 renamed FIFO_DATA3
- net D4 renamed FIFO_DATA4
- net D5 renamed FIFO_DATA5
- net D6 renamed FIFO_DATA6
- net FTDI_RD renamed FIFO_RD
- net FTDI_RXF renamed FIFO_RXF
- net FTDI_TXE renamed FIFO_TXE
- net FTDI_WR renamed FIFO_WR
- removed net D7: U1G$1.DATA7
- removed net FTDI_CLK6MHZ: U1G$1.CBUS6
- removed net FTDI_PWREN: U1G$1.CBUS5, U2.!EN1, U2.!EN2
- new net FIFO_CLK12MHZ: U1G$1.CBUS5
- new net FIFO_PWREN: R4.1, U1G$1.CBUS6, U2.!EN1, U2.!EN2
- new net N$2: R3.1, U1G$1.DATA7
- net 3V3_IN: now also C1.1, R4.2, U1G$1.!SIWU; no longer C3.1, U1G$1.!SI/WU
- net 5V_IN: now also C3.1; no longer C1.1
- net GND: now also R3.2
Other:
- note added: "Pull-up if programming FT240X in-circuit"

Commit message: Cleanup; add PoR and JTAG
Parts:
- added D1: (no value), led:LEDCHIP-LED0805
- added J2: JTAG, apple-idun:JTAG
- added J3: CON2X22, apple-idun:CON2X22
- added R5, R6, R7, R9: 100k, rcl:R-US_R0805
- added R8: 100, rcl:R-US_R0805
- added RESET: TACTSW, apple-idun:TACTSW
- R3, R4: value 100K -> 100k
Connections:
- net FIFO_CLK12MHZ renamed CLK12MHZ
- removed net FIFO_PWREN: R4.1, U1G$1.CBUS6, U2.!EN1, U2.!EN2
- new net A0: J3.W
- new net A1: J3.19
- new net A10: J3.R
- new net A11: J3.14
- new net A12: J3.P
- new net A13: J3.13
- new net A14: J3.N
- new net A15: J3.12
- new net A2: J3.V
- new net A3: J3.18
- new net A4: J3.U
- new net A5: J3.17
- new net A6: J3.T
- new net A7: J3.16
- new net A8: J3.S
- new net A9: J3.15
- new net D0: J3.9
- new net D1: J3.J
- new net D2: J3.8
- new net D3: J3.H
- new net D4: J3.7
- new net D5: J3.F
- new net D6: J3.6
- new net D7: J3.E
- new net IRQ: J3.4
- new net N$1: D1.C, R8.1
- new net NMI: J3.3
- new net PHI0: J3.M
- new net PHI1: J3.D
- new net PHI2: J3.A
- new net PWREN: R9.1, U1G$1.CBUS6, U2.!EN1, U2.!EN2
- new net R: J3.L
- new net RDY: J3.5
- new net RESET: J3.2, R7.2, RESET.2
- new net RW: J3.K
- new net S: J3.11
- new net SYNC: J3.B
- new net T: J3.21
- new net TCK: J2.TCK, R6.2
- new net TDI: J2.TDI
- new net TDO: J2.TDO
- new net TMS: J2.TMS
- net 3V3: now also J2.VREF, R6.1
- net 3V3_IN: now also C2.1, R9.2; no longer C1.1, R4.2
- net 5V: now also D1.A, J3.22, R7.1
- net 5V_IN: now also C1.1; no longer C2.1
- net FIFO_RD: now also R3.1
- net FIFO_WR: now also R4.1
- net GND: now also J2.GND, J3.20, J3.X, R4.2, R5.2, R8.2, RESET.1
- net N$2: now also R5.1; no longer R3.1
Other:
- note added: "!RF!/DMA/VMA/+12V/-12V NC"
- note added: "Assume original PoR behavior; manual pulse required after power-on"
- note added: "R9 required if programming FT240X in-circuit"
- note added: "REQUIRED MTP MEMORY CONFIGURATION Pull down I/O Pins in USB Suspend: Enabled Power Source: Bus Powered Max Bus Power Current: 500mA Load VCP Driver: Enabled CBUS5: CLK12MHz CBUS6: PWREN#"
- note added: "XC9500XL has internal pull-ups on TDI/TMS"
- note removed: "Pull-up if programming FT240X in-circuit"
