File: eagle/apple-mini.sch (EAGLE design)
At the start: 41 parts, among them J1 USBMICRO, J2 JTAG, J3 RBM22DRTN, U1 FT240XS, U2 SN74LVC2G17DBV, U3 TPS2082D, U4 MCS6502, U5 MC6821, U6 AS6C62256A, U7 AT28C64B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

Commit message: Route power and remaining critical nets
Connections:
- net A15: now also U8G$1.P38; no longer U8G$1.P36
- net CA1: now also U8G$1.P51; no longer U8G$1.P61
- net CA2: now also U8G$1.P56; no longer U8G$1.P62
- net DA: now also U8G$1.P39; no longer U8G$1.P47
- net FIFO_DATA0: now also U8G$1.P13; no longer U8G$1.P1
- net FIFO_DATA1: now also U8G$1.P9; no longer U8G$1.P2/GTS2
- net FIFO_DATA2: now also U8G$1.P11; no longer U8G$1.P4
- net FIFO_DATA3: now also U8G$1.P4; no longer U8G$1.P5/GTS1
- net FIFO_DATA4: now also U8G$1.P12; no longer U8G$1.P6
- net FIFO_DATA5: now also U8G$1.P6; no longer U8G$1.P7
- net FIFO_DATA6: now also U8G$1.P5/GTS1; no longer U8G$1.P8
- net FIFO_DATA7: now also U8G$1.P7; no longer U8G$1.P9
- net FIFO_RD: now also U8G$1.P2/GTS2; no longer U8G$1.P10
- net FIFO_RXF: now also U8G$1.P10; no longer U8G$1.P12
- net FIFO_TXE: now also U8G$1.P8; no longer U8G$1.P13
- net FIFO_WR: now also U8G$1.P1; no longer U8G$1.P11
- net GND: now also U8G$1.P20, U8G$1.P36, U8G$1.P62; no longer U8G$1.P31, U8G$1.P38, U8G$1.P50
- net PA0: now also U8G$1.P50; no longer U8G$1.P51
- net PA2: now also U8G$1.P57; no longer U8G$1.P56
- net PA3: now also U8G$1.P59; no longer U8G$1.P57
- net PA5: now also U8G$1.P60; no longer U8G$1.P59
- net PA6: now also U8G$1.P61; no longer U8G$1.P60
- net PB0: now also U8G$1.P47; no longer U8G$1.P39
- net PB1: now also U8G$1.P46; no longer U8G$1.P40
- net PB2: now also U8G$1.P45; no longer U8G$1.P42
- net PB3: now also U8G$1.P44; no longer U8G$1.P43
- net PB4: now also U8G$1.P43; no longer U8G$1.P44
- net PB5: now also U8G$1.P42; no longer U8G$1.P45
- net PB6: now also U8G$1.P40; no longer U8G$1.P46
- net PHI2: now also U8G$1.P19; no longer U8G$1.P32
- net R: now also U8G$1.P23; no longer U8G$1.P19
- net S: now also U8G$1.P22; no longer U8G$1.P20
- net T: now also U8G$1.P31; no longer U8G$1.P22
- net X: now also U8G$1.P32; no longer U8G$1.P23
- net Y: now also U8G$1.P25; no longer U8G$1.P24
- net Z: now also U8G$1.P24; no longer U8G$1.P25

Commit message: Initial (and incomplete) gerbers
Changed lines of the file:
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@@
 <?xml version="1.0" encoding="utf-8"?>
 <!DOCTYPE eagle SYSTEM "eagle.dtd">
-<eagle version="7.3.0">
+<eagle version="7.4.0">
 <drawing>
 <settings>
@@
 CBUS5: CLK12MHz
 CBUS6: PWREN#</text>
-<text x="104.14" y="40.64" size="1.27" layer="97" font="vector">50mA max</text>
-<text x="104.14" y="58.42" size="1.27" layer="97" font="vector">500mA max</text>
+<text x="104.14" y="40.64" size="1.27" layer="97" font="vector" ratio="10">50mA max</text>
+<text x="104.14" y="58.42" size="1.27" layer="97" font="vector" ratio="10">500mA max</text>
 </plain>
 <instances>
